Commit message: Removed torque_model from dynamixel_controller

File: deps/Robot_hybrid.urdf (robot description, URDF)
Before this commit: robot BipedalRobot, 15 links, 14 joints
Joints:
- joint base_boom_to_link_boom_joint_x: limit (none) -> lower=-1.57 upper=1.57
- joint world_to_base_boom_joint: limit (none) -> lower=-5.0 upper=5.0
